File: KiCad/Smartwatch.kicad_sch (KiCad schematic)
At the start: 96 parts, among them J1 5358, M1 LCM1027B3605F, Q1 AO3400A, SW1 SW_Push, SW2 JXTCONN TS-1010-S26, U1 BNO055, U10 Quectel LC76G, U11 MIC5504-1.8YM5, U12 ESP32-S3, U13 BMP280, U14 LD39100PU33R, U2 MIC5504-3.3YM5, U3 MAX30102, U4 MCP9808_DFN, U5 TPS2116DRL, U6 USBLC6-2SC6, U7 BRCL4054DME, U9 GC9A01_IPS_Display_w/_Touch, Y1 40MHz, Y2 32.768KHz, Y3 32.768KHz

Commit message: gonna jump off a builing on facebook live
Parts:
- added R16: 10k, Resistor_SMD:R_0402_1005Metric, symbol Device:R_Small
Connections:
- net GND: now also R16.2
- net GPSEN: now also R16.1
Changed lines of the file:
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@@
 	)
 	(junction
+		(at 234.95 26.67)
+		(diameter 0)
+		(color 0 0 0 0)
+	)
+	(junction
 		(at 163.83 60.96)
 		(diameter 0)
@@
 	(wire
 		(pts
+			(xy 234.95 26.67) (xy 237.49 26.67)
+		)
+		(stroke
+			(width 0)
+			(type default)
+		)
+	)
+	(wire
+		(pts
 			(xy 44.45 187.96) (xy 41.91 187.96)
 		)
@@
 	(wire
 		(pts
+			(xy 234.95 26.67) (xy 234.95 27.94)
+		)
+		(stroke
+			(width 0)
+			(type default)
+		)
+	)
+	(wire
+		(pts
 			(xy 73.66 20.32) (xy 86.36 20.32)
 		)
@@
 	(wire
 		(pts
-			(xy 227.33 26.67) (xy 237.49 26.67)
+			(xy 227.33 26.67) (xy 234.95 26.67)
 		)
 		(stroke
@@
 	)
 	(symbol
+		(lib_id "Device:R_Small")
+		(at 234.95 30.48 0)
+		(unit 1)
+		(exclude_from_sim no)
+		(in_bom yes)
+		(on_board yes)
+		(dnp no)
+		(property "Reference" "R16"
+			(at 236.982 29.972 0)
+			(effects
+				(font
+					(size 1.016 1.016)
+				)
+				(justify left)
+			)
+		)
+		(property "Value" "10k"
+			(at 236.728 31.75 0)
+			(effects
+				(font
+					(size 1.27 1.27)
+				)
+				(justify left)
+			)
+		)
+		(property "Footprint" "Resistor_SMD:R_0402_1005Metric"
+			(at 234.95 30.48 0)
+			(effects
+				(font
+					(size 1.27 1.27)
+				)
+				(hide yes)
+			)
+		)
+		(property "Datasheet" "~"
+			(at 234.95 30.48 0)
+			(effects
+				(font
+					(size 1.27 1.27)
+				)
+				(hide yes)
+			)
+		)
+		(property "Description" "Resistor, small symbol"
+			(at 234.95 30.48 0)
+			(effects
+				(font
+					(size 1.27 1.27)
+				)
+				(hide yes)
+			)
+		)
+		(pin "2"
+		)
+		(pin "1"
+		)
+		(instances
+			(project "Smartwatch"
+				(path "/e141b4c9-28fb-4bc3-aace-8a7adb0cdaa6"
+					(reference "R16")
+					(unit 1)
+				)
+			)
+		)
+	)
+	(symbol
 		(lib_id "power:+3.3V")
 		(at 30.48 43.18 0)
@@
 					(unit 1)
 				)
+			)
+		)
+	)
+	(symbol
+		(lib_id "power:GND")
+		(at 234.95 33.02 0)
+		(unit 1)
+		(exclude_from_sim no)
+		(in_bom yes)
+		(on_board yes)
+		(dnp no)
+		(property "Reference" "#PWR091"
+			(at 234.95 39.37 0)
+			(effects
+				(font
+					(size 1.27 1.27)
+				)
+				(hide yes)
+			)
+		)
+		(property "Value" "GND"
+			(at 234.95 36.576 0)
+			(effects
+				(font
+					(size 1.27 1.27)
+				)
+			)
+		)
+		(property "Footprint" ""
+			(at 234.95 33.02 0)
+			(effects
+				(font
+					(size 1.27 1.27)
+				)
+				(hide yes)
+			)
+		)
+		(property "Datasheet" ""
+			(at 234.95 33.02 0)
+			(effects
+				(font
+					(size 1.27 1.27)
+				)
+				(hide yes)
+			)
+		)
+		(property "Description" "Power symbol creates a global label with name \"GND\" , ground"
+			(at 234.95 33.02 0)
+			(effects
+				(font
+					(size 1.27 1.27)
+				)
+				(hide yes)
+			)
+		)
+		(pin "1"
+		)
+		(instances
+			(project "Smartwatch"
+				(path "/e141b4c9-28fb-4bc3-aace-8a7adb0cdaa6"
+					(reference "#PWR091")
+					(unit 1)
+				)

Commit message: changed up PCB design, still WIP
Parts:
- U12: Field5 Order ESP32-S3R8 If Possible -> Order ESP32-S3FH4R2 If Possible
Changed lines of the file:
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@@
 		(on_board yes)
 		(dnp no)
-		(fields_autoplaced yes)
 		(property "Reference" "SW1"
-			(at 232.41 35.56 0)
+			(at 232.41 38.608 0)
 			(effects
 				(font
@@
 					(size 1.27 1.27)
 				)
+				(hide yes)
 			)
 		)
@@
 			)
 		)
-		(property "Field5" "Order ESP32-S3R8 If Possible"
-			(at 139.7 150.368 0)
+		(property "Field5" "Order ESP32-S3FH4R2 If Possible"
+			(at 140.462 150.368 0)
 			(effects
 				(font
@@
 		(dnp no)
 		(property "Reference" "SW2"
-			(at 233.68 57.15 0)
+			(at 233.68 59.944 0)
 			(effects
 				(font
@@
 					(size 1.27 1.27)
 				)
+				(hide yes)
 			)
 		)
