File: KiCad/Smartwatch.kicad_sch (KiCad schematic)
At the start: 96 parts, among them J1 5358, M1 LCM1027B3605F, Q1 AO3400A, SW1 SW_Push, SW2 SW_Push, U1 BNO055, U10 Quectel LC76G, U11 MIC5504-1.8YM5, U12 ESP32-S3, U13 BMP280, U14 LD39100PU33R, U2 MIC5504-3.3YM5, U3 MAX30102, U4 MCP9808_DFN, U5 TPS2116DRL, U6 USBLC6-2SC6, U7 BRCL4054DME, U9 GC9A01_IPS_Display_w/_Touch, Y1 40MHz, Y2 32.768KHz, Y3 32.768KHz

Commit message: PCB V1
Parts:
- SW1: footprint (none) -> Usermade:JXTCONN TS-1010-S26
- SW2: value SW_Push -> JXTCONN TS-1010-S26; footprint (none) -> Usermade:JXTCONN TS-1010-S26
- U10: footprint (none) -> Usermade:quectel lc76g
- Y2, Y3: footprint (none) -> Usermade:EPSON Q13FC13500004
Connections:
- net GND: now also C19.1, R21.2, R22.2; no longer C19.2, R21.1, R22.1
- net at U1.6 (PS0): now also R21.1; no longer R21.2
- net at U1.5 (PS1): now also R22.1; no longer R22.2
- net at U1.9 (CAP): now also C19.2; no longer C19.1
Other:
- moved on the sheet: C19, R21, R22
Changed lines of the file:
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@@
 			)
 		)
-		(property "Footprint" ""
+		(property "Footprint" "Usermade:JXTCONN TS-1010-S26"
 			(at 232.41 38.1 0)
 			(effects
@@
 			)
 		)
-		(property "Footprint" ""
+		(property "Footprint" "Usermade:EPSON Q13FC13500004"
 			(at 138.43 177.8 0)
 			(effects
@@
 	(symbol
 		(lib_id "Device:R_Small")
-		(at 62.23 90.17 270)
+		(at 62.23 90.17 90)
+		(mirror x)
 		(unit 1)
 		(exclude_from_sim no)
@@
 		(dnp no)
 		(property "Reference" "R21"
-			(at 60.452 86.36 90)
+			(at 64.008 86.36 90)
 			(effects
 				(font
@@
 		)
 		(property "Value" "10k"
-			(at 60.452 88.392 90)
+			(at 64.008 88.392 90)
 			(effects
 				(font
@@
 	(symbol
 		(lib_id "Device:R_Small")
-		(at 62.23 92.71 270)
+		(at 62.23 92.71 90)
+		(mirror x)
 		(unit 1)
 		(exclude_from_sim no)
@@
 		(dnp no)
 		(property "Reference" "R22"
-			(at 68.326 91.44 90)
+			(at 56.134 91.44 90)
 			(effects
 				(font
@@
 		)
 		(property "Value" "10k"
-			(at 68.326 93.472 90)
+			(at 56.134 93.472 90)
 			(effects
 				(font
@@
 			)
 		)
-		(property "Footprint" ""
+		(property "Footprint" "Usermade:quectel lc76g"
 			(at 222.25 104.14 0)
 			(effects
@@
 			)
 		)
-		(property "Footprint" ""
+		(property "Footprint" "Usermade:EPSON Q13FC13500004"
 			(at 62.23 76.2 0)
 			(effects
@@
 	(symbol
 		(lib_id "Device:C_Small")
-		(at 62.23 95.25 90)
+		(at 62.23 95.25 270)
+		(mirror x)
 		(unit 1)
 		(exclude_from_sim no)
@@
 		(dnp no)
 		(property "Reference" "C19"
-			(at 60.452 99.568 90)
+			(at 64.008 99.568 90)
 			(effects
 				(font
@@
 		)
 		(property "Value" "100n"
-			(at 59.944 98.044 90)
+			(at 64.516 98.044 90)
 			(effects
 				(font
@@
 		(lib_id "Device:C_Small")
 		(at 212.09 54.61 0)
+		(mirror y)
 		(unit 1)
 		(exclude_from_sim no)
@@
 		(dnp no)
 		(property "Reference" "C22"
-			(at 214.376 53.34 0)
+			(at 209.804 53.34 0)
 			(effects
 				(font
@@
 		)
 		(property "Value" "10u"
-			(at 214.376 55.626 0)
+			(at 209.804 55.626 0)
 			(effects
 				(font
@@
 		(on_board yes)
 		(dnp no)
-		(fields_autoplaced yes)
 		(property "Reference" "SW2"
 			(at 233.68 57.15 0)
@@
 			)
 		)
-		(property "Value" "SW_Push"
-			(at 233.68 59.69 0)
+		(property "Value" "JXTCONN TS-1010-S26"
+			(at 233.426 67.056 0)
 			(effects
 				(font
@@
 			)
 		)
-		(property "Footprint" ""
+		(property "Footprint" "Usermade:JXTCONN TS-1010-S26"
 			(at 233.68 59.69 0)
 			(effects
@@
 					(size 1.27 1.27)
 				)
-				(hide yes)
 			)
 		)

Commit message: a lot of pcb updates, more to come
Parts:
- removed C29: 10u, Capacitor_SMD:C_0603_1608Metric, symbol Device:C_Small
- removed C30, C36: 100n, Capacitor_SMD:C_0402_1005Metric, symbol Device:C_Small
- added R16: 10k, Resistor_SMD:R_0402_1005Metric, symbol Device:R_Small
- JP1: footprint Connector_PinHeader_1.00mm:PinHeader_1x02_P1.00mm_Vertical -> Jumper:SolderJumper-2_P1.3mm_Open_RoundedPad1.0x1.5mm
- U12: Field5 Order ESP32-S3R8 If Possible -> Order ESP32-S3FH4R2 If Possible
Connections:
- net GND: now also R16.2
- net GPSEN: now also R16.1
