File: KiCad/Smartwatch.kicad_sch (KiCad schematic)
At the start: 96 parts, among them J1 5358, M1 LCM1027B3605F, Q1 AO3400A, SW1 SW_Push, SW2 SW_Push, U1 BNO055, U10 Quectel LC76G, U11 MIC5504-1.8YM5, U12 ESP32-S3, U13 BMP280, U14 LD39100PU33R, U2 MIC5504-3.3YM5, U3 MAX30102, U4 MCP9808_DFN, U5 TPS2116DRL, U6 USBLC6-2SC6, U7 BRCL4054DME, U9 GC9A01_IPS_Display_w/_Touch, Y1 40MHz, Y2 32.768KHz, Y3 32.768KHz

Commit message: final version of pcb
Parts:
- removed C29: 10u, Capacitor_SMD:C_0603_1608Metric, symbol Device:C_Small
- removed C30, C36: 100n, Capacitor_SMD:C_0402_1005Metric, symbol Device:C_Small
- added R16: 10k, Resistor_SMD:R_0402_1005Metric, symbol Device:R_Small
- JP1: footprint Connector_PinHeader_1.00mm:PinHeader_1x02_P1.00mm_Vertical -> Jumper:SolderJumper-2_P1.3mm_Open_RoundedPad1.0x1.5mm
- SW1: footprint (none) -> Usermade:JXTCONN TS-1010-S26
- SW2: value SW_Push -> JXTCONN TS-1010-S26; footprint (none) -> Usermade:JXTCONN TS-1010-S26
- U10: footprint (none) -> Usermade:quectel lc76g
- U12: Field5 Order ESP32-S3R8 If Possible -> Order ESP32-S3FH4R2 If Possible
- Y2, Y3: footprint (none) -> Usermade:EPSON Q13FC13500004
Connections:
- net GND: now also C19.1, R21.2, R22.2, R16.2; no longer C19.2, R21.1, R22.1
- net GPSEN: now also R16.1
- net at U1.6 (PS0): now also R21.1; no longer R21.2
- net at U1.5 (PS1): now also R22.1; no longer R22.2
- net at U1.9 (CAP): now also C19.2; no longer C19.1
Other:
- moved on the sheet: C19, R21, R22
