File: KiCad/Smartwatch.kicad_pcb (KiCad board)
At the start: 4 copper layers, 38.5 x 38.5 mm, 96 parts, among them J1 5358, M1 LCM1027B3605F, Q1 AO3400A, SW1 SW_Push, SW2 JXTCONN TS-1010-S26, U1 BNO055, U10 Quectel LC76G, U11 MIC5504-1.8YM5, U12 ESP32-S3, U13 BMP280, U14 LD39100PU33R, U2 MIC5504-3.3YM5, U3 MAX30102, U4 MCP9808_DFN, U5 TPS2116DRL, U6 USBLC6-2SC6, U7 BRCL4054DME, U9 GC9A01_IPS_Display_w/_Touch, Y1 40MHz, Y2 32.768KHz, Y3 32.768KHz

Commit message: minor updates - practice pulling to local branch
Connections:
- C19 pad 1: Net-(U1-CAP) -> GND
- C19 pad 2: GND -> Net-(U1-CAP)
- R21 pad 1: GND -> Net-(U1-PS0)
- R21 pad 2: Net-(U1-PS0) -> GND
- R22 pad 1: GND -> Net-(U1-PS1)
- R22 pad 2: Net-(U1-PS1) -> GND
Routing:
- net /CS: track 25.4 -> 22.1 mm
- net /MISO: track 16.8 -> 16.2 mm

Commit message: a lot of pcb updates, more to come
Parts:
- removed C29: 10u, Capacitor_SMD:C_0603_1608Metric
- removed C30, C36: 100n, Capacitor_SMD:C_0402_1005Metric
- added R16: 10k, Resistor_SMD:R_0402_1005Metric, F.Cu at (129.2, 101.2)
- AE2, C17, C18, C19, C2, C21, C25, C3, C33, C34, C35, C38, C4, C5, C7, C8, C9, J1, L2, R11, R12, R13, R19, R20, R22, R24, R25, U1, U10, U14, U2, U4, U7, Y2: moved to F.Cu
- C31, C32, R17, R18, Y3: moved to B.Cu
- JP1: footprint Connector_PinHeader_1.00mm:PinHeader_1x02_P1.00mm_Vertical -> Jumper:SolderJumper-2_P1.3mm_Open_RoundedPad1.0x1.5mm
- moved AE1 34.9 mm to (156.5, 97.6), turned to 75 degrees
- moved SW1 31.4 mm to (123.7, 89.6), turned to 67 degrees
- moved R22 31.2 mm to (156.9, 87.8), turned to 0 degrees
- moved SW2 31.2 mm to (124.5, 99.1), turned to 110 degrees
- moved C21 31.2 mm to (156.9, 89.7), turned to 0 degrees
- moved R19 30.9 mm to (156.9, 88.8), turned to 0 degrees
- moved C28 29.5 mm to (150.8, 96.0), turned to -135 degrees
- moved Y2 29.1 mm to (155.2, 93.8), turned to 180 degrees
- moved J1 29.0 mm to (135.8, 81.1)
- moved C17 28.8 mm to (156.2, 92.8), turned to 90 degrees
- moved AE2 28.1 mm to (149.2, 107.2), turned to 30 degrees
- moved C20 28.1 mm to (156.8, 90.7), turned to 0 degrees
- moved R21 27.9 mm to (155.9, 85.6), turned to 90 degrees
- moved R9 27.7 mm to (124.7, 96.3), turned to 110 degrees
- moved R5 27.6 mm to (125.7, 87.8), turned to 67 degrees
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Routing:
- net +3.3V: track 158.5 -> 40.9 mm, vias 24 -> 8
- net +3.3VGPS: track 32.3 -> 5.81 mm, vias 2 -> 0
- net /BAT_REF: track 25.2 -> 0.95 mm, vias 5 -> 0
- net /SDA: track 35.4 -> 58.8 mm, vias 4 -> 3
- net /CS: track 22.1 -> 0.00 mm, vias 1 -> 0
- net /LCD_BK: track 21.2 -> 0.00 mm, vias 2 -> 0
- net /LATCH: track 20.5 -> 0.00 mm, vias 2 -> 0
- net /MOSI: track 19.7 -> 0.00 mm, vias 1 -> 0
- net /MISO: track 16.2 -> 0.00 mm, vias 1 -> 0
- net /SCLK: track 15.9 -> 0.00 mm, vias 1 -> 0
- net /TX: track 6.48 -> 20.9 mm, vias 1 -> 2
- net /BT_2: track 16.3 -> 1.87 mm, vias 2 -> 0
- net /GPIO0: track 18.2 -> 4.77 mm, vias 2 -> 0
- net /CHRG_ST2: track 13.5 -> 0.00 mm, vias 2 -> 0
- net /TP_INT: track 12.7 -> 0.00 mm
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- added copper zone on In1.Cu, net +3.3V
- removed copper zone on In1.Cu, net GND
Other:
- board text added: "+-"
- board text added: "BOOT"
- board text added: "M"

Commit message: final traces hopfully
Parts:
- C13, C14: moved to B.Cu
- moved C23 5.34 mm to (134.7, 94.0)
- moved C2 5.03 mm to (147.0, 80.5), turned to 0 degrees
- moved C24 1.93 mm to (135.9, 92.1), turned to 90 degrees
- moved C14 1.59 mm to (132.5, 93.5)
- moved C13 1.43 mm to (137.5, 89.5), turned to 0 degrees
- moved Y3 0.94 mm to (134.9, 86.2)
- moved C32 0.88 mm to (136.5, 86.0)
- moved C31 0.81 mm to (133.0, 89.5)
- moved C12 0.71 mm to (142.0, 98.0), turned to -135 degrees
- moved JP1 0.25 mm to (143.6, 88.0)
- moved R27 0.22 mm to (134.7, 89.4)
Routing:
- net /LCD_BK: track 0.00 -> 67.1 mm, vias 0 -> 7
- net /CHRG_ST2: track 0.00 -> 56.9 mm, vias 0 -> 5
- net /LCD_RST: track 0.00 -> 51.3 mm, vias 0 -> 2
- net /LCD_DC: track 0.00 -> 47.4 mm, vias 0 -> 2
- net /BAT_REF: track 0.95 -> 40.2 mm, vias 0 -> 4
- net /VIBE: track 4.70 -> 43.0 mm, vias 0 -> 8
- net /TP_INT: track 0.00 -> 37.8 mm, vias 0 -> 3
- net +3.3V: track 40.9 -> 76.8 mm, vias 8 -> 14
- net /CS: track 0.00 -> 31.2 mm, vias 0 -> 2
- net /SCLK: track 0.00 -> 28.2 mm, vias 0 -> 2
- net /CHRG_ST: track 0.00 -> 27.6 mm, vias 0 -> 6
- net /MOSI: track 0.00 -> 25.6 mm, vias 0 -> 1
- net /INT_BNO: track 0.00 -> 25.1 mm, vias 0 -> 4
- net /~{INT}_MAX: track 1.18 -> 23.9 mm, vias 0 -> 1
- net /BATV: track 11.3 -> 33.8 mm, vias 0 -> 2
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