File: KiCad/Smartwatch.kicad_pcb (KiCad board)
At the start: 4 copper layers, 38.5 x 38.5 mm, 95 parts, among them J1 5358, M1 LCM1027B3605F, Q1 AO3400A, SW1 SW_Push, SW2 JXTCONN TS-1010-S26, U1 BNO055, U10 Quectel LC76G, U11 MIC5504-1.8YM5, U12 ESP32-S3, U13 BMP280, U14 LD39100PU33R, U2 MIC5504-3.3YM5, U3 MAX30102, U4 MCP9808_DFN, U5 TPS2116DRL, U6 USBLC6-2SC6, U7 BRCL4054DME, U9 GC9A01_IPS_Display_w/_Touch, Y1 40MHz, Y2 32.768KHz, Y3 32.768KHz

Commit message: Names Added
Other:
- board text added: "Argel Romano"
- board text added: "Jeffery Wong"
- board text added: "Jodelys Dejesus"
- board text added: "Laura Tolley"
- board text added: "Matthew Wilson"
- board text added: "Rebecca Duran"
- board text added: "Thabothan Varatharasa"
- board text added: "William Herr"
Changed lines of the file:
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@@
+		)
+	)
+	(gr_text "Jodelys Dejesus"
+		(at 137.403117 109.073046 0)
+		(layer "B.SilkS")
+		(effects
+			(font
+				(size 0.5 0.5)
+				(thickness 0.125)
+				(bold yes)
+			)
+			(justify left bottom mirror)
+		)
+	)
+	(gr_text "Matthew Wilson"
+		(at 138.177414 105.113902 0)
+		(layer "B.SilkS")
+		(effects
+			(font
+				(size 0.5 0.5)
+				(thickness 0.125)
+			)
+			(justify left bottom mirror)
+		)
+	)
+	(gr_text "Thabothan Varatharasa"
+		(at 138.089758 108.240311 0)
+		(layer "B.SilkS")
+		(effects
+			(font
+				(size 0.5 0.5)
+				(thickness 0.125)
+				(bold yes)
+			)
+			(justify left bottom mirror)
+		)
+	)
+	(gr_text "Rebecca Duran"
+		(at 137.373898 109.891172 0)
+		(layer "B.SilkS")
+		(effects
+			(font
+				(size 0.5 0.5)
+				(thickness 0.125)
+				(bold yes)
+			)
+			(justify left bottom mirror)
+		)
+	)
+	(gr_text "Laura Tolley"
+		(at 138.031321 106.633278 0)
+		(layer "B.SilkS")
+		(effects
+			(font
+				(size 0.5 0.5)
+				(thickness 0.125)
+				(bold yes)
+			)
+			(justify left bottom mirror)
+		)
+	)
+	(gr_text "William Herr"
+		(at 138.206633 104.324995 0)
+		(layer "B.SilkS")
+		(effects
+			(font
+				(size 0.5 0.5)
+				(thickness 0.1)
+				(bold yes)
+			)
+			(justify left bottom mirror)
+		)
+	)
+	(gr_text "Argel Romano"
+		(at 138.089758 107.422185 0)
+		(layer "B.SilkS")
+		(effects
+			(font
+				(size 0.5 0.5)
+				(thickness 0.125)
+				(bold yes)
+			)
+			(justify left bottom mirror)
+		)
+	)
+	(gr_text "Jeffery Wong "
+		(at 138.016711 105.858981 0)
+		(layer "B.SilkS")
+		(effects
+			(font
+				(size 0.5 0.5)
+				(thickness 0.125)
+				(bold yes)
+			)
+			(justify left bottom mirror)
 		)
 	)
